File: AstraDriverPCB/AstraDriver.kicad_sch (KiCad schematic)
At the start: 2 parts

Commit message: Progress
Parts:
- removed R1, R2: 10, LiveAstra:R_0402_1005Metric, symbol LiveAstra:R_10Ohm_0402_62mW
Connections:
- no-connect marks 1 -> 0
Other:
- added sheet Block Diagram (block_diagram.kicad_sch)
- added sheet Overview (overview.kicad_sch)
- note added: "23 June 2024"
- note added: "4 Channel LED Driver with PWM dimming input. LED2001PHR is the driver IC, it can support up to 4A, 3V - 18V at 850KHz switching frequency."
- note added: "4 PWM channels"
- note added: "5V and 3.3V Power Input"
- note added: "AstraDriver"
- note added: "Features"
- note added: "In review"
- note added: "JST VH Connectors"
- note added: "Render for reference only"
- company: (none) -> LiveAstra Technologies
