File: AstraDriverPCB/led_driver_blue_cy_2A5.kicad_sch (KiCad schematic)
At the start: 7 parts, among them U1 LED2001PHR

Commit message: Prepare for review, cleanup
Parts:
- removed INF3: ~, symbol LiveAstra:Information_Box_XL
- added INF2: ~, symbol LiveAstra:Information_Box_XL
- renumbered C4 to C3, C5 to C4, C6 to C5, R7 to R12

Commit message: Cleanup
Parts:
- renumbered INF2 to INF3
Other:
- note added: "Blue and CY"
Changed lines of the file:
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@@
+		)
+	)
+	(text "Blue and CY"
+		(exclude_from_sim no)
+		(at 25.4 25.4 0)
+		(effects
+			(font
+				(face "ING Me Headline")
+				(size 8 8)
+			)
+			(justify left top)
 		)
 	)
@@
 		(dnp no)
 		(fields_autoplaced yes)
-		(property "Reference" "INF2"
+		(property "Reference" "INF3"
 			(at 179.07 27.9399 0)
 			(effects
@@
 			(project "AstraDriver"
 				(path "/d8760d88-6646-4dd8-a980-02e776803cc5/db9d16fd-00a9-4695-9dd4-6de80f9e2ffc/02378fe8-1086-45ec-8926-c2e9ee784828"
-					(reference "INF2")
-					(unit 1)
-				)
-				(path "/d8760d88-6646-4dd8-a980-02e776803cc5/db9d16fd-00a9-4695-9dd4-6de80f9e2ffc/2917a49e-0b0c-4bc9-a147-180770b18779"
 					(reference "INF3")
 					(unit 1)
 				)
+				(path "/d8760d88-6646-4dd8-a980-02e776803cc5/db9d16fd-00a9-4695-9dd4-6de80f9e2ffc/2917a49e-0b0c-4bc9-a147-180770b18779"
+					(reference "INF4")
+					(unit 1)
+				)
