File: AstraDriverPCB/AstraDriver.kicad_pcb (KiCad board)
At the start: 4 copper layers, 102 x 65 mm, 113 parts, among them CN1 JST VH 8 PIN, CN2 JST VH 2 PIN, CN3 JST VH 2 PIN, CN4 JST VH 2 PIN, CN5 JST VH 2 PIN, CN6 JST VH 2 PIN, U1 LED2001PHR, U2 LED2001PHR, U3 LED2001PHR, U4 LED2001PHR

Commit message: Layout complete
Parts:
- removed kibuzzard-672641C9: G***, kibuzzard-672641C9
- removed kibuzzard-672641CE: G***, kibuzzard-672641CE
- removed kibuzzard-67264513: G***, kibuzzard-67264513
- removed kibuzzard-6726451B: G***, kibuzzard-6726451B
- removed kibuzzard-67264761: G***, kibuzzard-67264761
- removed kibuzzard-6726476F: G***, kibuzzard-6726476F
- removed kibuzzard-67264778: G***, kibuzzard-67264778
- removed kibuzzard-6726477C: G***, kibuzzard-6726477C
- removed kibuzzard-6762FA53: G***, kibuzzard-6762FA53
- added kibuzzard-67B1DE0F: G***, kibuzzard-67B1DE0F, B.Cu at (131.2, 73.0)
- added kibuzzard-67B1DE14: G***, kibuzzard-67B1DE14, B.Cu at (126.5, 73.0)
- added kibuzzard-67B1DE99: G***, kibuzzard-67B1DE99, B.Cu at (173.5, 115.5)
- added kibuzzard-67B1DE99: G***, kibuzzard-67B1DE99, B.Cu at (137.5, 115.5)
- added kibuzzard-67B1DE99: G***, kibuzzard-67B1DE99, B.Cu at (155.5, 115.5)
- added kibuzzard-67B1DE99: G***, kibuzzard-67B1DE99, B.Cu at (119.5, 115.5)
- added kibuzzard-67B1DEA2: G***, kibuzzard-67B1DEA2, B.Cu at (123.5, 115.5)
- added kibuzzard-67B1DEA2: G***, kibuzzard-67B1DEA2, B.Cu at (141.5, 115.5)
- added kibuzzard-67B1DEA2: G***, kibuzzard-67B1DEA2, B.Cu at (177.5, 115.5)
- added kibuzzard-67B1DEA2: G***, kibuzzard-67B1DEA2, B.Cu at (159.5, 115.5)
- added kibuzzard-67B1DFB0: G***, kibuzzard-67B1DFB0, F.Cu at (116.2, 77.5)
- added kibuzzard-67B1DFC8: G***, kibuzzard-67B1DFC8, F.Cu at (116.2, 73.2)
- kibuzzard-67264EAC, kibuzzard-67264F3E, kibuzzard-67264F60, kibuzzard-67264F65: moved to B.Cu
- moved kibuzzard-67264F65 73.5 mm to (166.2, 101.8)
- moved kibuzzard-67264F3E 71.2 mm to (166.2, 105.0)
- moved kibuzzard-67264EAC 62.2 mm to (131.0, 105.0)
- moved kibuzzard-67264F60 60.2 mm to (131.0, 101.8)
- moved TP2 9.50 mm to (182.8, 81.5)
- moved TP8 9.50 mm to (173.2, 81.5)
Routing:
- net /Block Diagram/RSRV: track 8.56 -> 15.3 mm, vias 1 -> 0
- net GND: vias 157 -> 198

Commit message: SLK tweaks
Parts:
- added kibuzzard-67EB9EA5: G***, kibuzzard-67EB9EA5, F.Cu at (116.0, 72.5)
- added kibuzzard-67EB9FE0: G***, kibuzzard-67EB9FE0, F.Cu at (182.8, 72.5)
- moved kibuzzard-67B1DFB0 66.5 mm to (182.8, 77.5)
- moved kibuzzard-67B1DFC8 4.25 mm to (116.2, 77.5)

Commit message: Tweaks
Routing:
- net GND: vias 198 -> 196
- net +5V: vias 34 -> 30
